File: Hardware/pcb final v5.brd (EAGLE design)
At the start: 170.2 x 111.2 mm, 103 parts, among them IC1 BD5229G-TR, IC4 XC6220A331MR-G, J1 FH34SRJ-24S-0.5SH_99_, J2 SAMACSYS_PARTS_USB4110-GF-A, J3 QWIIC_RIGHT_ANGLE, J4 112A-TAAR-R03_ATTEND, Q1 20V/4.2A/52mΩ/1.4W, Q2 20V/4.2A/52mΩ/1.4W, Q3 SI1308EDL-T1-GE3, U1 W25Q512JVEIQ, U2 ESP32-C6-WROOM-1-N8, U3 DS3231SN#, U4 MAX17048G+T10

Commit message: resolved issues
Routing:
- net 3V3: track 454.8 -> 457.4 mm
- net MISO: track 83.7 -> 84.7 mm
Changed lines of the file:
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@@
 </via>
+<polygon width="0.1524" layer="1" spacing="1.27" pour="solid" thermals="yes">
+<vertex x="92.2646" y="10.0431625"/>
+<vertex x="92.2762" y="10.01515625"/>
+<vertex x="92.2762" y="0.0762"/>
+<vertex x="170.1238" y="0.0762"/>
+<vertex x="170.1238" y="67.1238"/>
+<vertex x="92.18484375" y="67.1238"/>
+<vertex x="92.1568375" y="67.1354"/>
+<vertex x="92.1354" y="67.1568375"/>
+<vertex x="92.1238" y="67.18484375"/>
+<vertex x="92.1238" y="111.1238"/>
+<vertex x="68.0762" y="111.1238"/>
+<vertex x="68.0762" y="110.18484375"/>
+<vertex x="68.0646" y="110.1568375"/>
+<vertex x="68.0431625" y="110.1354"/>
+<vertex x="68.01515625" y="110.1238"/>
+<vertex x="19.68484375" y="110.1238"/>
+<vertex x="19.6568375" y="110.1354"/>
+<vertex x="19.6354" y="110.1568375"/>
+<vertex x="19.6238" y="110.18484375"/>
+<vertex x="19.6238" y="111.1238"/>
+<vertex x="0.0762" y="111.1238"/>
+<vertex x="0.0762" y="65.7762"/>
+<vertex x="6.31515625" y="65.7762"/>
+<vertex x="6.3431625" y="65.7646"/>
+<vertex x="6.3646" y="65.7431625"/>
+<vertex x="6.3762" y="65.71515625"/>
+<vertex x="6.3762" y="47.68484375"/>
+<vertex x="6.3646" y="47.6568375"/>
+<vertex x="6.3431625" y="47.6354"/>
+<vertex x="6.31515625" y="47.6238"/>
+<vertex x="0.0762" y="47.6238"/>
+<vertex x="0.0762" y="0.0762"/>
+<vertex x="73.9238" y="0.0762"/>
+<vertex x="73.9238" y="10.01515625"/>
+<vertex x="73.9354" y="10.0431625"/>
+<vertex x="73.9568375" y="10.0646"/>
+<vertex x="73.98484375" y="10.0762"/>
+<vertex x="92.21515625" y="10.0762"/>
+<vertex x="92.2431625" y="10.0646"/>
+</polygon>
+<polygon width="0.1524" layer="16" spacing="1.27" pour="solid" thermals="yes">
+<vertex x="92.2646" y="10.0431625"/>
+<vertex x="92.2762" y="10.01515625"/>
+<vertex x="92.2762" y="0.0762"/>
+<vertex x="170.1238" y="0.0762"/>
+<vertex x="170.1238" y="67.1238"/>
+<vertex x="92.18484375" y="67.1238"/>
+<vertex x="92.1568375" y="67.1354"/>
+<vertex x="92.1354" y="67.1568375"/>
+<vertex x="92.1238" y="67.18484375"/>
+<vertex x="92.1238" y="111.1238"/>
+<vertex x="68.0762" y="111.1238"/>
+<vertex x="68.0762" y="110.18484375"/>
+<vertex x="68.0646" y="110.1568375"/>
+<vertex x="68.0431625" y="110.1354"/>
+<vertex x="68.01515625" y="110.1238"/>
+<vertex x="19.68484375" y="110.1238"/>
+<vertex x="19.6568375" y="110.1354"/>
+<vertex x="19.6354" y="110.1568375"/>
+<vertex x="19.6238" y="110.18484375"/>
+<vertex x="19.6238" y="111.1238"/>
+<vertex x="0.0762" y="111.1238"/>
+<vertex x="0.0762" y="65.7762"/>
+<vertex x="6.31515625" y="65.7762"/>
+<vertex x="6.3431625" y="65.7646"/>
+<vertex x="6.3646" y="65.7431625"/>
+<vertex x="6.3762" y="65.71515625"/>
+<vertex x="6.3762" y="47.68484375"/>
+<vertex x="6.3646" y="47.6568375"/>
+<vertex x="6.3431625" y="47.6354"/>
+<vertex x="6.31515625" y="47.6238"/>
+<vertex x="0.0762" y="47.6238"/>
+<vertex x="0.0762" y="0.0762"/>
+<vertex x="73.9238" y="0.0762"/>
+<vertex x="73.9238" y="10.01515625"/>
+<vertex x="73.9354" y="10.0431625"/>
+<vertex x="73.9568375" y="10.0646"/>
+<vertex x="73.98484375" y="10.0762"/>
+<vertex x="92.21515625" y="10.0762"/>
+<vertex x="92.2431625" y="10.0646"/>
+</polygon>
 <polygon width="0.1524" layer="1" spacing="1.27" pour="solid" thermals="yes">
 <vertex x="6.3646" y="47.6568375"/>
@@
 <wire x1="60.386" y1="108.861" x2="60.39" y2="108.8578" width="0.3" layer="1"/>
 <wire x1="52.69925" y1="108.861" x2="52.6" y2="108.8578" width="0.3" layer="1"/>
-<wire x1="42.17325" y1="95.7035" x2="42.17325" y2="59.6935" width="0.3" layer="1"/>
-<wire x1="47.57475" y1="101.105" x2="42.17325" y2="95.7035" width="0.3" layer="1"/>
+<wire x1="42.17325" y1="95.7035" x2="42.17325" y2="93.65" width="0.3" layer="1"/>
+<wire x1="42.17325" y1="93.65" x2="42.17325" y2="59.6935" width="0.3" layer="1"/>
+<wire x1="47.57475" y1="101.105" x2="44.059875" y2="97.590125" width="0.3" layer="1"/>
+<wire x1="44.059875" y1="97.590125" x2="42.17325" y2="95.7035" width="0.3" layer="1"/>
 <wire x1="47.85175" y1="101.105" x2="47.57475" y2="101.105" width="0.3" layer="1"/>
 <wire x1="42.17325" y1="59.6935" x2="42.104" y2="59.555" width="0.3" layer="1"/>
@@
 <wire x1="21.1905" y1="107.26825" x2="21.1905" y2="108.03" width="0.3" layer="1"/>
 <wire x1="32.686" y1="95.77275" x2="21.1905" y2="107.26825" width="0.3" layer="1"/>
-<wire x1="42.03475" y1="95.77275" x2="32.686" y2="95.77275" width="0.3" layer="1"/>
+<wire x1="32.686" y1="95.77275" x2="39.85" y2="95.77275" width="0.3" layer="1"/>
 <wire x1="20.498" y1="108.7225" x2="20.38" y2="108.8578" width="0.3" layer="1"/>
-<wire x1="42.03475" y1="95.77275" x2="42.17325" y2="95.7035" width="0.3" layer="1"/>
 <wire x1="13.64225" y1="43.00425" x2="19.113" y2="43.00425" width="0.3" layer="1"/>
 <wire x1="9.07175" y1="47.57475" x2="13.64225" y2="43.00425" width="0.3" layer="1"/>
@@
 <wire x1="5.4015" y1="90.302" x2="5.738215625" y2="90.426040625" width="0.3" layer="1"/>
 <wire x1="9.0025" y1="48.12875" x2="9.01" y2="47.99" width="0.3" layer="1"/>
+<wire x1="39.85" y1="95.77275" x2="41.667375" y2="97.590125" width="0.3" layer="1"/>
+<wire x1="41.667375" y1="97.590125" x2="44.059875" y2="97.590125" width="0.3" layer="1"/>
 </signal>
 <signal name="N$10">
@@
 <wire x1="34.902" y1="57.96225" x2="34.902" y2="57.7545" width="0.15" layer="1"/>
 <wire x1="36.35625" y1="59.4165" x2="34.902" y2="57.96225" width="0.15" layer="1"/>
-<wire x1="36.35625" y1="62.67125" x2="36.35625" y2="59.4165" width="0.15" layer="1"/>
+<wire x1="36.35625" y1="61.65" x2="36.35625" y2="59.4165" width="0.15" layer="1"/>
 <wire x1="39.40325" y1="65.71825" x2="36.35625" y2="62.67125" width="0.15" layer="1"/>
 <wire x1="34.902" y1="57.7545" x2="34.895" y2="57.695" width="0.15" layer="1"/>
@@
 <wire x1="9.8335" y1="97.98875" x2="9.8335" y2="97.29625" width="0.15" layer="1"/>
 <wire x1="5.9555" y1="93.7645" x2="5.955490625" y2="93.724946875" width="0.15" layer="1"/>
-<wire x1="9.0025" y1="94.734" x2="9.0025" y2="74.85925" width="0.15" layer="1"/>
-<wire x1="9.0025" y1="74.85925" x2="9.0025" y2="65.5105" width="0.15" layer="1"/>
+<wire x1="9.0025" y1="94.734" x2="9.0025" y2="76.15" width="0.15" layer="1"/>
+<wire x1="9.0025" y1="76.15" x2="9.0025" y2="65.5105" width="0.15" layer="1"/>
 <wire x1="8.136875" y1="95.599625" x2="9.0025" y2="94.734" width="0.15" layer="1"/>
 <wire x1="9.0025" y1="65.5105" x2="9.01" y2="65.49" width="0.15" layer="1"/>
-<wire x1="28.60025" y1="62.67125" x2="36.35625" y2="62.67125" width="0.15" layer="1"/>
+<wire x1="28.60025" y1="62.67125" x2="35.35" y2="62.67125" width="0.15" layer="1"/>
+<wire x1="35.35" y1="62.67125" x2="36.35625" y2="62.67125" width="0.15" layer="1"/>
 <wire x1="16.41225" y1="74.85925" x2="28.60025" y2="62.67125" width="0.15" layer="1"/>
-<wire x1="9.0025" y1="74.85925" x2="16.41225" y2="74.85925" width="0.15" layer="1"/>
+<wire x1="10.29325" y1="74.85925" x2="16.41225" y2="74.85925" width="0.15" layer="1"/>
+<wire x1="9.0025" y1="76.15" x2="10.29325" y2="74.85925" width="0.15" layer="1"/>
+<wire x1="35.35" y1="62.67125" x2="36.35625" y2="61.665" width="0.15" layer="1"/>
+<wire x1="36.35625" y1="61.665" x2="36.35625" y2="61.65" width="0.15" layer="1"/>
 </signal>
 <signal name="RESET">
@@
 <signal name="N$2">
 </signal>
+<signal name="N$3">
+</signal>
 </signals>
 <mfgpreviewcolors>
@@
 will not be understood (or retained) with this version.
 </note>
-<note version="8.3" severity="warning">
-Since Version 8.3, EAGLE supports the association of 3D packages
-with devices in libraries, schematics, and board files. Those 3D
-packages will not be understood (or retained) with this version.
-</note>
 </compatibility>
